File: hardware/hardware.kicad_sch (KiCad schematic)
At the start: 61 parts, among them J1 BATT, J10 Trk next, J11 Trk prev, J12 Vol up, J13 Vol down, J14 Reset, J2 RFID-RC522, J3 104031-0811, J4 PROG, J5 EXT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

Commit message: kosmetik
Parts:
- J10: footprint (none) -> Connector_PinHeader_2.54mm:PinHeader_1x02_P2.54mm_Vertical
Changed lines of the file:
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@@
+    (stroke (width 0) (type default) (color 0 0 0 0))
+  )
+  (wire (pts (xy 251.46 97.79) (xy 251.46 106.68))
     (stroke (width 0) (type default) (color 0 0 0 0))
   )
@@
   )
   (wire (pts (xy 40.64 118.11) (xy 25.4 118.11))
-    (stroke (width 0) (type default) (color 0 0 0 0))
-  )
-  (wire (pts (xy 251.46 97.79) (xy 251.46 106.68))
     (stroke (width 0) (type default) (color 0 0 0 0))
   )
@@
     (property "Reference" "J10" (id 0) (at 23.495 170.18 0))
     (property "Value" "Trk next" (id 1) (at 23.495 167.64 0))
-    (property "Footprint" "" (id 2) (at 24.13 162.56 0)
-      (effects (font (size 1.27 1.27)) hide)
-    )
+    (property "Footprint" "Connector_PinHeader_2.54mm:PinHeader_1x02_P2.54mm_Vertical" (id 2) (at 24.13 162.56 0)
+      (effects (font (size 1.27 1.27)) hide)
+    )
